File: SnarkBarkerMCA.sch (KiCad schematic (older format))
At the start: 177 parts, among them J1 BUS_MCA, J2 HPLA_PORT, J3 Conn_01x06, J4 HPLA_PORT, J5 HPLA_PORT, J6 DEBUG, P1 Joystick/MIDI, T1 2N3904, T2 2N3904, U1 NE558, U10 YM3014B, U11 NJM3403A, U12 MC1408_DIP, U13 805X, U14 SAA1099, U15 SAA1099, U18 74HCT374, U19 74HCT374, U2 74HCT245, U20 74HCT74, U21 74HCT125, U22 74HCT74, U23 74HCT74, U24 74HCT32, U25 SPARE, U26 74HCT74, U27 74HCT32, U28 74HCT08, U29 74HCT14, U3 74HCT244, U30 74HCT32, U31 XC9572XL-TQ100, U32 TC1262-3.3V, U5 LM324, U6 LM393, U9 YM3812

Commit message: Combine R41 into R26,R39 line item
Parts:
- R41: symbol Device:R -> Device:R_Small
Changed lines of the file:
@@
 $EndComp
 $Comp
-L Device:R R41
+L Device:R_Small R41
 U 1 1 5C1A2681
 P 5550 13500
-F 0 "R41" V 5630 13500 50  0000 C CNN
-F 1 "4.7K" V 5550 13500 50  0000 C CNN
+F 0 "R41" H 5800 13550 50  0000 C CNN
+F 1 "4.7K" H 5800 13450 50  0000 C CNN
 F 2 "SoundBlaster:SB_R_AXIAL_400" V 5480 13500 50  0001 C CNN
 F 3 "" H 5550 13500 50  0001 C CNN
@@
 Connection ~ 5450 14050
 Wire Wire Line
-	5550 14050 5550 13650
+	5550 14050 5550 13600
 Wire Wire Line
 	4700 14150 4550 14150
@@
 Connection ~ 6750 11850
 Wire Wire Line
-	5550 13300 5550 13350
+	5550 13300 5550 13400
 Wire Wire Line
 	7550 14600 7550 14700

Commit message: Logic chip update
Parts:
- U18, U19: value 74HCT374 -> 74AHCT374; Mouser 595-SN74HCT374N -> 595-SN74AHCT374N
- U2: value 74HCT245 -> 74AHCT245; Mouser 595-SN74HCT245NE4 -> 595-SN74AHCT245N
- U20, U22, U23, U26: value 74HCT74 -> 74AHCT74; Mouser 595-SN74HCT74NE4 -> 595-SN74AHCT74N
- U21: value 74HCT125 -> 74AHCT125; Mouser 595-SN74HCT125NE4 -> 595-SN74AHCT125N
- U24, U27, U30: value 74HCT32 -> 74AHCT32; Mouser 595-SN74HCT32NE4 -> 595-SN74AHCT32N
- U28: value 74HCT08 -> 74AHCT08; Mouser 595-SN74HCT08NE4 -> 595-SN74AHCT08N
- U29: value 74HCT14 -> 74AHCT14; Mouser 595-SN74HCT14N -> 595-SN74AHCT14N
- U3: value 74HCT244 -> 74AHCT244; Mouser 595-SN74HCT244NE4 -> 595-SN74AHCT244N
